File: CNC_interface.sch (KiCad schematic (older format))
At the start: 25 parts, among them J1 Conn_01x04_Male, J10 Conn_01x08, J11 Conn_01x08, J12 Conn_01x08, J13 Conn_01x08, J14 Conn_01x03_Male, J15 Conn_01x03_Male, J16 Conn_01x03_Male, J2 Conn_01x04_Male, J3 Conn_01x04_Male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

Commit message: adding capacitance footprints
Parts:
- C1: footprint (none) -> Capacitor_THT:CP_Radial_D8.0mm_P3.50mm
- C2: footprint (none) -> Capacitor_THT:CP_Radial_D10.0mm_P5.00mm
Changed lines of the file:
@@
 F 0 "C1" H 7268 5496 50  0000 L CNN
 F 1 "CP" H 7268 5405 50  0000 L CNN
-F 2 "" H 7188 5300 50  0001 C CNN
+F 2 "Capacitor_THT:CP_Radial_D8.0mm_P3.50mm" H 7188 5300 50  0001 C CNN
 F 3 "~" H 7150 5450 50  0001 C CNN
 	1    7150 5450
@@
 F 0 "C2" H 4018 5496 50  0000 L CNN
 F 1 "CP" H 4018 5405 50  0000 L CNN
-F 2 "" H 3938 5300 50  0001 C CNN
+F 2 "Capacitor_THT:CP_Radial_D10.0mm_P5.00mm" H 3938 5300 50  0001 C CNN
 F 3 "~" H 3900 5450 50  0001 C CNN
 	1    3900 5450
